File: hardware/gate-rail/gate-rail.kicad_pcb (KiCad board)
At the start: 2 copper layers, 224 x 15 mm, 22 parts, among them J1 IDC-Header_2x05_P2.54mm_Verti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, Q1 LED_D3.0mm, Q2 LED_D3.0mm, Q3 LED_D3.0mm, Q4 LED_D3.0mm, Q5 LED_D3.0mm, Q6 LED_D3.0mm

Commit message: Gate-rail: fix 62 schematic-parity issues (metadata sync)
The rail board carried raw library footprint identities: gen_rail_pcb.py's
placement loop set only ref + pad nets, never FPID / Value / LCSC / Variant. So
every D/Q/R showed value "LED_D5.0mm" instead of "IR333C-A", bare footprint names
missing the library nickname, and no LCSC/Variant fields -> 41 mismatch + 19 field
+ 2 extra_footprint (H1/H2).

Fixes (mirroring the driver's gen_pcb.py place_all):
- load_netlist() now also reads <value> + LCSC + Variant fields into a meta map.
- Placement loop sets SetFPID(LIB_ID) + SetValue + SetField("LCSC"/"Variant"),
  keeping LCSC/Variant HIDDEN (SetField defaults to visible on silk -> was adding
  ~69 silk overlaps; hidden restores the 20-warning baseline).
- H1/H2 mounting holes flagged SetBoardOnly + SetExcludedFromBOM (exempt from
  extra_footprint parity), matching the driver.
- TP1 symbol marked in_bom=False so its exclude-from-BOM matches the footprint.

Result: kicad-cli --schematic-parity 0 / 0 electrical / 0 unconnected; ERC 0;
validate.py --production PASS; station-spacing assertion PASS; variant BOMs
regenerated (EMIT 13, RECV 7). Fully deterministic, no autorouter.

Co-Authored-By: Claude Opus 4.8 <noreply@anthropic.com>
Parts:
- D1, D2, D3, D4, D5, D6: value LED_D5.0mm -> IR333C-A; footprint LED_D5.0mm -> LED_THT:LED_D5.0mm
- J1: value IDC-Header_2x05_P2.54mm_Vertical -> RAIL-IDC; footprint IDC-Header_2x05_P2.54mm_Vertical -> Connector_IDC:IDC-Header_2x05_P2.54mm_Vertical
- Q1, Q2, Q3, Q4, Q5, Q6: value LED_D3.0mm -> PT204-6B; footprint LED_D3.0mm -> LED_THT:LED_D3.0mm
- R1, R2, R3, R4, R5, R6: value R_0603_1608Metric -> 150; footprint R_0603_1608Metric -> Resistor_SMD:R_0603_1608Metric
- TP1: value TestPoint_Pad_1.5x1.5mm -> SIG_SPARE; footprint TestPoint_Pad_1.5x1.5mm -> TestPoint:TestPoint_Pad_1.5x1.5mm
