File: hardware/omnimarble-driver/boost_charger.kicad_sch (KiCad schematic)
At the start: 44 parts, among them K1 HF3FF-12V, K2 HF3FF-12V, Q1 MMBT3904, Q2 MMBT3904, Q3 MMBT3904, Q91 AOD66923, U4 UC3843B, U5 TL431B

Commit message: Snapshot driver's final validated state before parking as vNext
Fold the last regeneration into the repo so the source is internally consistent
with the already-committed board/BOM (the Q90 diode->MOSFET fix + JLC cart
substitutions previously landed only in the root schematic + board):
- 7 driver schematic sub-sheets, regenerated to carry the final part numbers.
- fab/jlc/ORDER_NOTES.md — final BOM (J2/J5 C707836, R21/R22 C5110275, etc.).
- omnimarble-driver-5-rev-39.ses — the routing session import-clean rebuilds the
  board from; committing it keeps the routed board reproducible while parked.

Timestamp-only gerber/zip churn and scratch (.ses iterations, drc/erc reports,
logs) were left out. Driver stays vNext/on-hold per V0_BENCH_RIG.md.

Co-Authored-By: Claude Opus 4.8 <noreply@anthropic.com>
Parts:
- R21, R22: LCSC C216413 -> C5110275
- U4: LCSC C16414 -> C2995531
