File: hardware/omnimarble-driver/mcu_status.kicad_sch (KiCad schematic)
At the start: 10 parts, among them J10 PICO-SOCKET, J9 PICO-SOCKET, Q4 MMBT3904

Commit message: Snapshot driver's final validated state before parking as vNext
Fold the last regeneration into the repo so the source is internally consistent
with the already-committed board/BOM (the Q90 diode->MOSFET fix + JLC cart
substitutions previously landed only in the root schematic + board):
- 7 driver schematic sub-sheets, regenerated to carry the final part numbers.
- fab/jlc/ORDER_NOTES.md — final BOM (J2/J5 C707836, R21/R22 C5110275, etc.).
- omnimarble-driver-5-rev-39.ses — the routing session import-clean rebuilds the
  board from; committing it keeps the routed board reproducible while parked.

Timestamp-only gerber/zip churn and scratch (.ses iterations, drc/erc reports,
logs) were left out. Driver stays vNext/on-hold per V0_BENCH_RIG.md.

Co-Authored-By: Claude Opus 4.8 <noreply@anthropic.com>
Parts:
- D15: LCSC C72043 -> C2289
Changed lines of the file:
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@@
 		(instances
 			(project "omnimarble-driver"
-				(path "/4f6b9534-97fd-44ae-b81e-62754cb6cba6/75f25778-acbd-42b3-9f04-352847a17f55"
+				(path "/e983a447-c241-422e-9650-13442643de66/c52f051a-2bda-4f95-9ce1-e3fc3b41d38d"
 					(reference "J9")
 					(unit 1)
@@
 		(instances
 			(project "omnimarble-driver"
-				(path "/4f6b9534-97fd-44ae-b81e-62754cb6cba6/75f25778-acbd-42b3-9f04-352847a17f55"
+				(path "/e983a447-c241-422e-9650-13442643de66/c52f051a-2bda-4f95-9ce1-e3fc3b41d38d"
 					(reference "J10")
 					(unit 1)
@@
 		(instances
 			(project "omnimarble-driver"
-				(path "/4f6b9534-97fd-44ae-b81e-62754cb6cba6/75f25778-acbd-42b3-9f04-352847a17f55"
+				(path "/e983a447-c241-422e-9650-13442643de66/c52f051a-2bda-4f95-9ce1-e3fc3b41d38d"
 					(reference "R70")
 					(unit 1)
@@
 		(instances
 			(project "omnimarble-driver"
-				(path "/4f6b9534-97fd-44ae-b81e-62754cb6cba6/75f25778-acbd-42b3-9f04-352847a17f55"
+				(path "/e983a447-c241-422e-9650-13442643de66/c52f051a-2bda-4f95-9ce1-e3fc3b41d38d"
 					(reference "D14")
 					(unit 1)
@@
 		(instances
 			(project "omnimarble-driver"
-				(path "/4f6b9534-97fd-44ae-b81e-62754cb6cba6/75f25778-acbd-42b3-9f04-352847a17f55"
+				(path "/e983a447-c241-422e-9650-13442643de66/c52f051a-2bda-4f95-9ce1-e3fc3b41d38d"
 					(reference "R71")
 					(unit 1)
@@
 			)
 		)
-		(property "LCSC" "C72043"
+		(property "LCSC" "C2289"
 			(at 229.87 80.01 0)
 			(show_name no)
@@
 		(instances
 			(project "omnimarble-driver"
-				(path "/4f6b9534-97fd-44ae-b81e-62754cb6cba6/75f25778-acbd-42b3-9f04-352847a17f55"
+				(path "/e983a447-c241-422e-9650-13442643de66/c52f051a-2bda-4f95-9ce1-e3fc3b41d38d"
 					(reference "D15")
 					(unit 1)
@@
 		(instances
 			(project "omnimarble-driver"
-				(path "/4f6b9534-97fd-44ae-b81e-62754cb6cba6/75f25778-acbd-42b3-9f04-352847a17f55"
+				(path "/e983a447-c241-422e-9650-13442643de66/c52f051a-2bda-4f95-9ce1-e3fc3b41d38d"
 					(reference "Q4")
 					(unit 1)
@@
 		(instances
 			(project "omnimarble-driver"
-				(path "/4f6b9534-97fd-44ae-b81e-62754cb6cba6/75f25778-acbd-42b3-9f04-352847a17f55"
+				(path "/e983a447-c241-422e-9650-13442643de66/c52f051a-2bda-4f95-9ce1-e3fc3b41d38d"
 					(reference "R72")
 					(unit 1)
@@
 		(instances
 			(project "omnimarble-driver"
-				(path "/4f6b9534-97fd-44ae-b81e-62754cb6cba6/75f25778-acbd-42b3-9f04-352847a17f55"
+				(path "/e983a447-c241-422e-9650-13442643de66/c52f051a-2bda-4f95-9ce1-e3fc3b41d38d"
 					(reference "BZ1")
 					(unit 1)
@@
 		(instances
 			(project "omnimarble-driver"
-				(path "/4f6b9534-97fd-44ae-b81e-62754cb6cba6/75f25778-acbd-42b3-9f04-352847a17f55"
+				(path "/e983a447-c241-422e-9650-13442643de66/c52f051a-2bda-4f95-9ce1-e3fc3b41d38d"
 					(reference "D16")
 					(unit 1)
@@
 		(instances
 			(project "omnimarble-driver"
-				(path "/4f6b9534-97fd-44ae-b81e-62754cb6cba6/75f25778-acbd-42b3-9f04-352847a17f55"
+				(path "/e983a447-c241-422e-9650-13442643de66/c52f051a-2bda-4f95-9ce1-e3fc3b41d38d"
 					(reference "#PWR0016")
 					(unit 1)
