File: hardware/omnimarble-driver/power_input.kicad_sch (KiCad schematic)
At the start: 18 parts, among them J1 24V-IN, Q90 AOD4185, U1 AP63205, U2 78L12, U3 MCP6002

Commit message: Address external design review: boost FB + OVP redesign, BOM freeze
Review findings accepted and fixed (each verified by machine check):

1. Boost feedback network was wrong (confirmed: as-drawn spanned
   54-68V with PWM inverted vs the comment). Redesigned: RT/RB/RJ =
   100k/10k/9.1k with the exact transfer function documented in the
   schematic and design-calcs.md. PWM=0 (MCU-dead state) commands
   55.0V; full PWM commands 18.7V (below the 24.5V converter floor).
   New calcs.py asserts both endpoints.
2. OVP tripped at 55.6V, not the claimed 63V (confirmed). Redesigned:
   CJ431 (+/-0.5%) + 100k/4.3k 1% -> 60.5V nominal, 59.1-62.0V across
   tolerances. Protection ladder asserted in calcs.py: 55V operating
   < 59.1V trip-min, 62.0V trip-max < 63V cap rating - 1V. Operating
   ceiling deliberately reduced 60->55V to keep the bands disjoint.
3. BOM/schematic controller split-brain: bom.csv was stale
   (pre-UC3843 swap); regenerated from parts.py. Both now UC3843B.
4. High-power placeholders now real orderable parts (LCSC-verified):
   47R/5W SQM cement C5807995, dump redesigned to 2x 100R/10W cement
   in series C216413 (no 20-25W part stocked on LCSC; 5.3s to <5V),
   50mR/3W 2512 C2994645, 63V/35V electrolytics C28241/C176666, 10uH
   Sunlord C79272, MINI fuses+Keystone 3568 holders, buzzer, Pico
   sockets/breakout headers. Single documented exception: the 6.8k/2W
   bleed (CRH2512J6K80E04Z) is marked ORDER-REVIEW because LCSC's
   search is uncrawlable - validate.py allowlists it visibly.
5. validate.py pulled forward from the fab phase: fails on unknown
   footprints, blank LCSC on machine-placed parts, missing Variant
   fields, and duplicate refs; generates per-variant gate-rail BOMs
   (bom_rail_emit/recv.csv). Caught two bad footprint names.
6. Paralleling constraints now on the schematic (same-lot FETs,
   symmetric copper, <25mm gate loops, driver return at shunt star).
7. Fail-safe defaults hardened: MCU_FIRE and FIRE_GATED get explicit
   pulldow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
Parts:
- C1: footprint Capacitor_SMD:CP_Elec_10x10.5 -> Capacitor_SMD:CP_Elec_6.3x7.7; LCSC (none) -> C176666
- F1: LCSC (none) -> C5249699
- L1: footprint Inductor_SMD:L_12x12mm_H8mm -> Inductor_SMD:L_Changjiang_FNR6045S; LCSC (none) -> C79272
Changed lines of the file:
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@@
 		(instances
 			(project "omnimarble-driver"
-				(path "/73d8eff6-39f1-4e5f-a80b-a36699d4dd7c/fa789c71-1167-4558-bca0-71f763939438"
+				(path "/324ed851-0be4-493c-900d-5ec8847c0520/1c05de07-b56e-4659-a9ed-186313cc062a"
 					(reference "J1")
 					(unit 1)
@@
 			)
 		)
+		(property "LCSC" "C5249699"
+			(at 69.85 44.45 0)
+			(show_name no)
+			(do_not_autoplace no)
+			(hide yes)
+			(effects
+				(font
+					(size 1.27 1.27)
+				)
+			)
+		)
 		(pin "1"
 		)
@@
 		(instances
 			(project "omnimarble-driver"
-				(path "/73d8eff6-39f1-4e5f-a80b-a36699d4dd7c/fa789c71-1167-4558-bca0-71f763939438"
+				(path "/324ed851-0be4-493c-900d-5ec8847c0520/1c05de07-b56e-4659-a9ed-186313cc062a"
 					(reference "F1")
 					(unit 1)
@@
 		(instances
 			(project "omnimarble-driver"
-				(path "/73d8eff6-39f1-4e5f-a80b-a36699d4dd7c/fa789c71-1167-4558-bca0-71f763939438"
+				(path "/324ed851-0be4-493c-900d-5ec8847c0520/1c05de07-b56e-4659-a9ed-186313cc062a"
 					(reference "Q90")
 					(unit 1)
@@
 		(instances
 			(project "omnimarble-driver"
-				(path "/73d8eff6-39f1-4e5f-a80b-a36699d4dd7c/fa789c71-1167-4558-bca0-71f763939438"
+				(path "/324ed851-0be4-493c-900d-5ec8847c0520/1c05de07-b56e-4659-a9ed-186313cc062a"
 					(reference "R1")
 					(unit 1)
@@
 		(instances
 			(project "omnimarble-driver"
-				(path "/73d8eff6-39f1-4e5f-a80b-a36699d4dd7c/fa789c71-1167-4558-bca0-71f763939438"
+				(path "/324ed851-0be4-493c-900d-5ec8847c0520/1c05de07-b56e-4659-a9ed-186313cc062a"
 					(reference "D1")
 					(unit 1)
@@
 		(instances
 			(project "omnimarble-driver"
-				(path "/73d8eff6-39f1-4e5f-a80b-a36699d4dd7c/fa789c71-1167-4558-bca0-71f763939438"
+				(path "/324ed851-0be4-493c-900d-5ec8847c0520/1c05de07-b56e-4659-a9ed-186313cc062a"
 					(reference "D90")
 					(unit 1)
@@
 			)
 		)
-		(property "Footprint" "Capacitor_SMD:CP_Elec_10x10.5"
+		(property "Footprint" "Capacitor_SMD:CP_Elec_6.3x7.7"
 			(at 149.86 49.53 0)
 			(show_name no)
@@
 			)
 		)
+		(property "LCSC" "C176666"
+			(at 149.86 49.53 0)
+			(show_name no)
+			(do_not_autoplace no)
+			(hide yes)
+			(effects
+				(font
+					(size 1.27 1.27)
+				)
+			)
+		)
 		(pin "1"
 		)
@@
 		(instances
 			(project "omnimarble-driver"
-				(path "/73d8eff6-39f1-4e5f-a80b-a36699d4dd7c/fa789c71-1167-4558-bca0-71f763939438"
+				(path "/324ed851-0be4-493c-900d-5ec8847c0520/1c05de07-b56e-4659-a9ed-186313cc062a"
 					(reference "C1")
 					(unit 1)
@@
 		(instances
 			(project "omnimarble-driver"
-				(path "/73d8eff6-39f1-4e5f-a80b-a36699d4dd7c/fa789c71-1167-4558-bca0-71f763939438"
+				(path "/324ed851-0be4-493c-900d-5ec8847c0520/1c05de07-b56e-4659-a9ed-186313cc062a"
 					(reference "U1")
 					(unit 1)
@@
 		(instances
 			(project "omnimarble-driver"
-				(path "/73d8eff6-39f1-4e5f-a80b-a36699d4dd7c/fa789c71-1167-4558-bca0-71f763939438"
+				(path "/324ed851-0be4-493c-900d-5ec8847c0520/1c05de07-b56e-4659-a9ed-186313cc062a"
 					(reference "C2")
 					(unit 1)
@@
 			)
 		)
-		(property "Footprint" "Inductor_SMD:L_12x12mm_H8mm"
+		(property "Footprint" "Inductor_SMD:L_Changjiang_FNR6045S"
 			(at 100.33 115.57 0)
 			(show_name no)
@@
 			)
 		)
+		(property "LCSC" "C79272"
+			(at 100.33 115.57 0)
+			(show_name no)
+			(do_not_autoplace no)
+			(hide yes)
+			(effects
+				(font
+					(size 1.27 1.27)
+				)
+			)
+		)
 		(pin "1"
 		)
@@
 		(instances
 			(project "omnimarble-driver"
-				(path "/73d8eff6-39f1-4e5f-a80b-a36699d4dd7c/fa789c71-1167-4558-bca0-71f763939438"
+				(path "/324ed851-0be4-493c-900d-5ec8847c0520/1c05de07-b56e-4659-a9ed-186313cc062a"
 					(reference "L1")
 					(unit 1)
@@
 		(instances
 			(project "omnimarble-driver"
-				(path "/73d8eff6-39f1-4e5f-a80b-a36699d4dd7c/fa789c71-1167-4558-bca0-71f763939438"
+				(path "/324ed851-0be4-493c-900d-5ec8847c0520/1c05de07-b56e-4659-a9ed-186313cc062a"
 					(reference "C3")
 					(unit 1)
@@
 		(instances
 			(project "omnimarble-driver"
-				(path "/73d8eff6-39f1-4e5f-a80b-a36699d4dd7c/fa789c71-1167-4558-bca0-71f763939438"
+				(path "/324ed851-0be4-493c-900d-5ec8847c0520/1c05de07-b56e-4659-a9ed-186313cc062a"
 					(reference "C4")
 					(unit 1)
@@
 		(instances
 			(project "omnimarble-driver"
-				(path "/73d8eff6-39f1-4e5f-a80b-a36699d4dd7c/fa789c71-1167-4558-bca0-71f763939438"
+				(path "/324ed851-0be4-493c-900d-5ec8847c0520/1c05de07-b56e-4659-a9ed-186313cc062a"
 					(reference "U2")
 					(unit 1)
@@
 		(instances
 			(project "omnimarble-driver"
-				(path "/73d8eff6-39f1-4e5f-a80b-a36699d4dd7c/fa789c71-1167-4558-bca0-71f763939438"
+				(path "/324ed851-0be4-493c-900d-5ec8847c0520/1c05de07-b56e-4659-a9ed-186313cc062a"
 					(reference "C5")
 					(unit 1)
@@
 		(instances
 			(project "omnimarble-driver"
-				(path "/73d8eff6-39f1-4e5f-a80b-a36699d4dd7c/fa789c71-1167-4558-bca0-71f763939438"
+				(path "/324ed851-0be4-493c-900d-5ec8847c0520/1c05de07-b56e-4659-a9ed-186313cc062a"
 					(reference "C6")
 					(unit 1)
@@
 		(instances
 			(project "omnimarble-driver"
-				(path "/73d8eff6-39f1-4e5f-a80b-a36699d4dd7c/fa789c71-1167-4558-bca0-71f763939438"
+				(path "/324ed851-0be4-493c-900d-5ec8847c0520/1c05de07-b56e-4659-a9ed-186313cc062a"
 					(reference "R2")
 					(unit 1)
@@
 		(instances
 			(project "omnimarble-driver"
-				(path "/73d8eff6-39f1-4e5f-a80b-a36699d4dd7c/fa789c71-1167-4558-bca0-71f763939438"
+				(path "/324ed851-0be4-493c-900d-5ec8847c0520/1c05de07-b56e-4659-a9ed-186313cc062a"
 					(reference "R3")
 					(unit 1)
@@
 		(instances
 			(project "omnimarble-driver"
-				(path "/73d8eff6-39f1-4e5f-a80b-a36699d4dd7c/fa789c71-1167-4558-bca0-71f763939438"
+				(path "/324ed851-0be4-493c-900d-5ec8847c0520/1c05de07-b56e-4659-a9ed-186313cc062a"
 					(reference "U3")
 					(unit 2)
@@
 		(instances
 			(project "omnimarble-driver"
-				(path "/73d8eff6-39f1-4e5f-a80b-a36699d4dd7c/fa789c71-1167-4558-bca0-71f763939438"
+				(path "/324ed851-0be4-493c-900d-5ec8847c0520/1c05de07-b56e-4659-a9ed-186313cc062a"
 					(reference "#FLG0001")
 					(unit 1)
@@
 		(instances
 			(project "omnimarble-driver"
-				(path "/73d8eff6-39f1-4e5f-a80b-a36699d4dd7c/fa789c71-1167-4558-bca0-71f763939438"
+				(path "/324ed851-0be4-493c-900d-5ec8847c0520/1c05de07-b56e-4659-a9ed-186313cc062a"
 					(reference "#FLG0002")
 					(unit 1)
@@
 		(instances
 			(project "omnimarble-driver"
-				(path "/73d8eff6-39f1-4e5f-a80b-a36699d4dd7c/fa789c71-1167-4558-bca0-71f763939438"
+				(path "/324ed851-0be4-493c-900d-5ec8847c0520/1c05de07-b56e-4659-a9ed-186313cc062a"
 					(reference "#PWR0003")
 					(unit 1)
@@
 		(instances
 			(project "omnimarble-driver"
-				(path "/73d8eff6-39f1-4e5f-a80b-a36699d4dd7c/fa789c71-1167-4558-bca0-71f763939438"
+				(path "/324ed851-0be4-493c-900d-5ec8847c0520/1c05de07-b56e-4659-a9ed-186313cc062a"
 					(reference "#FLG0004")
 					(unit 1)
@@
 		(instances
 			(project "omnimarble-driver"
-				(path "/73d8eff6-39f1-4e5f-a80b-a36699d4dd7c/fa789c71-1167-4558-bca0-71f763939438"
+				(path "/324ed851-0be4-493c-900d-5ec8847c0520/1c05de07-b56e-4659-a9ed-186313cc062a"
 					(reference "#FLG0005")
 					(unit 1)
@@
 		(instances
 			(project "omnimarble-driver"
-				(path "/73d8eff6-39f1-4e5f-a80b-a36699d4dd7c/fa789c71-1167-4558-bca0-71f763939438"
+				(path "/324ed851-0be4-493c-900d-5ec8847c0520/1c05de07-b56e-4659-a9ed-186313cc062a"
 					(reference "#FLG0006")
 					(unit 1)
@@
 		(instances
 			(project "omnimarble-driver"
-				(path "/73d8eff6-39f1-4e5f-a80b-a36699d4dd7c/fa789c71-1167-4558-bca0-71f763939438"
+				(path "/324ed851-0be4-493c-900d-5ec8847c0520/1c05de07-b56e-4659-a9ed-186313cc062a"
 					(reference "#PWR0007")
 					(unit 1)

Commit message: Driver PCB: resolve both safety blockers + should-fixes, re-route, DRC-clean
Two datasheet-level blockers (invisible to netlist checks) + the should-fixes
from two review rounds, then a full DeepPCB re-route on the corrected netlist.

Blockers:
- U5 shunt ref: CJ431/C3113 (pinout 1=REF,2=K,3=A) did NOT match the TL431DBZ
  footprint -> OVP dead. Now TL431BIDBZR/C41283 (+/-0.5%, 1=K,2=REF,3=A). Kept
  +/-0.5% grade (the 1% A-grade would blow the 62.0V OVP ceiling).
- Relay HF3FF footprint had NO/NC transposed (datasheet bottom-view copied
  without mirroring) -> dump/charge logic inverted. Swapped pads 12<->14 +
  corrected silk. VERIFY WITH OHMMETER at bring-up (COM-NC @rest) -- parity is
  green by construction, DRC cannot see this.

Should-fixes: D90 SMBJ33A->SMBJ26CA (bidirectional, clamps below AP63205);
snubber 4.7k->4.7Ohm; R7 0.05->0.15Ohm (boost ilim); R25 10k->47k (0.28W->0.06W
LED series); BZ1 polarity swap. 78L12->DPAK deferred (reflows the placement
band; documented, fan-cool for bench per user).

Routing: full DeepPCB re-route from the corrected DSN. dsn_fixup now injects a
B.Cu keepout over the FET-strip corridor so the router can't pack signals where
the SHUNT_HI bus lives (rev-40 dropped the locked bus). import-clean re-authors
the SHUNT_HI B.Cu bus deterministically. Post-import repairs: re-authored the
RS1->NT1 Kelvin tie (DeepPCB routed SHUNT_HI on F.Cu shorting ISNS_P), joined a
MCU_FIRE via gap, bulged GATE6 off a 3V3 via, island-removal + a stitch via to
unify the fragmented F.Cu SHUNT_HI pour.

DRC 0 electrical / 0 unconnected; validate.py --production, validate_widths,
check_netlist, calcs all PASS.

Co-Authored-By: Claude Opus 4.8 <noreply@anthropic.com>
Parts:
- D90: value SMBJ33A -> SMBJ26CA; LCSC C19077586 -> C113996
Changed lines of the file:
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@@
 		(instances
 			(project "omnimarble-driver"
-				(path "/3eaa9588-078e-48af-b393-9dad6bd20142/62eeab2e-1b72-4517-8983-437fbddb3cf0"
+				(path "/4f6b9534-97fd-44ae-b81e-62754cb6cba6/78b057db-20e0-48a6-a5e1-06c21da7677d"
 					(reference "J1")
 					(unit 1)
@@
 		(instances
 			(project "omnimarble-driver"
-				(path "/3eaa9588-078e-48af-b393-9dad6bd20142/62eeab2e-1b72-4517-8983-437fbddb3cf0"
+				(path "/4f6b9534-97fd-44ae-b81e-62754cb6cba6/78b057db-20e0-48a6-a5e1-06c21da7677d"
 					(reference "F1")
 					(unit 1)
@@
 		(instances
 			(project "omnimarble-driver"
-				(path "/3eaa9588-078e-48af-b393-9dad6bd20142/62eeab2e-1b72-4517-8983-437fbddb3cf0"
+				(path "/4f6b9534-97fd-44ae-b81e-62754cb6cba6/78b057db-20e0-48a6-a5e1-06c21da7677d"
 					(reference "Q90")
 					(unit 1)
@@
 		(instances
 			(project "omnimarble-driver"
-				(path "/3eaa9588-078e-48af-b393-9dad6bd20142/62eeab2e-1b72-4517-8983-437fbddb3cf0"
+				(path "/4f6b9534-97fd-44ae-b81e-62754cb6cba6/78b057db-20e0-48a6-a5e1-06c21da7677d"
 					(reference "R1")
 					(unit 1)
@@
 		(instances
 			(project "omnimarble-driver"
-				(path "/3eaa9588-078e-48af-b393-9dad6bd20142/62eeab2e-1b72-4517-8983-437fbddb3cf0"
+				(path "/4f6b9534-97fd-44ae-b81e-62754cb6cba6/78b057db-20e0-48a6-a5e1-06c21da7677d"
 					(reference "D1")
 					(unit 1)
@@
 			)
 		)
-		(property "Value" "SMBJ33A"
+		(property "Value" "SMBJ26CA"
 			(at 134.62 82.55 0)
 			(show_name no)
@@
 			)
 		)
-		(property "LCSC" "C19077586"
+		(property "LCSC" "C113996"
 			(at 134.62 80.01 0)
 			(show_name no)
@@
 		(instances
 			(project "omnimarble-driver"
-				(path "/3eaa9588-078e-48af-b393-9dad6bd20142/62eeab2e-1b72-4517-8983-437fbddb3cf0"
+				(path "/4f6b9534-97fd-44ae-b81e-62754cb6cba6/78b057db-20e0-48a6-a5e1-06c21da7677d"
 					(reference "D90")
 					(unit 1)
@@
 		(instances
 			(project "omnimarble-driver"
-				(path "/3eaa9588-078e-48af-b393-9dad6bd20142/62eeab2e-1b72-4517-8983-437fbddb3cf0"
+				(path "/4f6b9534-97fd-44ae-b81e-62754cb6cba6/78b057db-20e0-48a6-a5e1-06c21da7677d"
 					(reference "C1")
 					(unit 1)
@@
 		(instances
 			(project "omnimarble-driver"
-				(path "/3eaa9588-078e-48af-b393-9dad6bd20142/62eeab2e-1b72-4517-8983-437fbddb3cf0"
+				(path "/4f6b9534-97fd-44ae-b81e-62754cb6cba6/78b057db-20e0-48a6-a5e1-06c21da7677d"
 					(reference "U1")
 					(unit 1)
@@
 		(instances
 			(project "omnimarble-driver"
-				(path "/3eaa9588-078e-48af-b393-9dad6bd20142/62eeab2e-1b72-4517-8983-437fbddb3cf0"
+				(path "/4f6b9534-97fd-44ae-b81e-62754cb6cba6/78b057db-20e0-48a6-a5e1-06c21da7677d"
 					(reference "C2")
 					(unit 1)
@@
 		(instances
 			(project "omnimarble-driver"
-				(path "/3eaa9588-078e-48af-b393-9dad6bd20142/62eeab2e-1b72-4517-8983-437fbddb3cf0"
+				(path "/4f6b9534-97fd-44ae-b81e-62754cb6cba6/78b057db-20e0-48a6-a5e1-06c21da7677d"
 					(reference "L1")
 					(unit 1)
@@
 		(instances
 			(project "omnimarble-driver"
-				(path "/3eaa9588-078e-48af-b393-9dad6bd20142/62eeab2e-1b72-4517-8983-437fbddb3cf0"
+				(path "/4f6b9534-97fd-44ae-b81e-62754cb6cba6/78b057db-20e0-48a6-a5e1-06c21da7677d"
 					(reference "C3")
 					(unit 1)
@@
 		(instances
 			(project "omnimarble-driver"
-				(path "/3eaa9588-078e-48af-b393-9dad6bd20142/62eeab2e-1b72-4517-8983-437fbddb3cf0"
+				(path "/4f6b9534-97fd-44ae-b81e-62754cb6cba6/78b057db-20e0-48a6-a5e1-06c21da7677d"
 					(reference "C4")
 					(unit 1)
@@
 		(instances
 			(project "omnimarble-driver"
-				(path "/3eaa9588-078e-48af-b393-9dad6bd20142/62eeab2e-1b72-4517-8983-437fbddb3cf0"
+				(path "/4f6b9534-97fd-44ae-b81e-62754cb6cba6/78b057db-20e0-48a6-a5e1-06c21da7677d"
 					(reference "U2")
 					(unit 1)
@@
 		(instances
 			(project "omnimarble-driver"
-				(path "/3eaa9588-078e-48af-b393-9dad6bd20142/62eeab2e-1b72-4517-8983-437fbddb3cf0"
+				(path "/4f6b9534-97fd-44ae-b81e-62754cb6cba6/78b057db-20e0-48a6-a5e1-06c21da7677d"
 					(reference "C5")
 					(unit 1)
@@
 		(instances
 			(project "omnimarble-driver"
-				(path "/3eaa9588-078e-48af-b393-9dad6bd20142/62eeab2e-1b72-4517-8983-437fbddb3cf0"
+				(path "/4f6b9534-97fd-44ae-b81e-62754cb6cba6/78b057db-20e0-48a6-a5e1-06c21da7677d"
 					(reference "C6")
 					(unit 1)
@@
 		(instances
 			(project "omnimarble-driver"
-				(path "/3eaa9588-078e-48af-b393-9dad6bd20142/62eeab2e-1b72-4517-8983-437fbddb3cf0"
+				(path "/4f6b9534-97fd-44ae-b81e-62754cb6cba6/78b057db-20e0-48a6-a5e1-06c21da7677d"
 					(reference "R2")
 					(unit 1)
@@
 		(instances
 			(project "omnimarble-driver"
-				(path "/3eaa9588-078e-48af-b393-9dad6bd20142/62eeab2e-1b72-4517-8983-437fbddb3cf0"
+				(path "/4f6b9534-97fd-44ae-b81e-62754cb6cba6/78b057db-20e0-48a6-a5e1-06c21da7677d"
 					(reference "R3")
 					(unit 1)
@@
 		(instances
 			(project "omnimarble-driver"
-				(path "/3eaa9588-078e-48af-b393-9dad6bd20142/62eeab2e-1b72-4517-8983-437fbddb3cf0"
+				(path "/4f6b9534-97fd-44ae-b81e-62754cb6cba6/78b057db-20e0-48a6-a5e1-06c21da7677d"
 					(reference "U3")
 					(unit 2)
@@
 		(instances
 			(project "omnimarble-driver"
-				(path "/3eaa9588-078e-48af-b393-9dad6bd20142/62eeab2e-1b72-4517-8983-437fbddb3cf0"
+				(path "/4f6b9534-97fd-44ae-b81e-62754cb6cba6/78b057db-20e0-48a6-a5e1-06c21da7677d"
 					(reference "#FLG0001")
 					(unit 1)
@@
 		(instances
 			(project "omnimarble-driver"
-				(path "/3eaa9588-078e-48af-b393-9dad6bd20142/62eeab2e-1b72-4517-8983-437fbddb3cf0"
+				(path "/4f6b9534-97fd-44ae-b81e-62754cb6cba6/78b057db-20e0-48a6-a5e1-06c21da7677d"
 					(reference "#FLG0002")
 					(unit 1)
@@
 		(instances
 			(project "omnimarble-driver"
-				(path "/3eaa9588-078e-48af-b393-9dad6bd20142/62eeab2e-1b72-4517-8983-437fbddb3cf0"
+				(path "/4f6b9534-97fd-44ae-b81e-62754cb6cba6/78b057db-20e0-48a6-a5e1-06c21da7677d"
 					(reference "#PWR0003")
 					(unit 1)
@@
 		(instances
 			(project "omnimarble-driver"
-				(path "/3eaa9588-078e-48af-b393-9dad6bd20142/62eeab2e-1b72-4517-8983-437fbddb3cf0"
+				(path "/4f6b9534-97fd-44ae-b81e-62754cb6cba6/78b057db-20e0-48a6-a5e1-06c21da7677d"
 					(reference "#FLG0004")
 					(unit 1)
@@
 		(instances
 			(project "omnimarble-driver"
-				(path "/3eaa9588-078e-48af-b393-9dad6bd20142/62eeab2e-1b72-4517-8983-437fbddb3cf0"
+				(path "/4f6b9534-97fd-44ae-b81e-62754cb6cba6/78b057db-20e0-48a6-a5e1-06c21da7677d"
 					(reference "#FLG0005")
 					(unit 1)
@@
 		(instances
 			(project "omnimarble-driver"
-				(path "/3eaa9588-078e-48af-b393-9dad6bd20142/62eeab2e-1b72-4517-8983-437fbddb3cf0"
+				(path "/4f6b9534-97fd-44ae-b81e-62754cb6cba6/78b057db-20e0-48a6-a5e1-06c21da7677d"
 					(reference "#FLG0006")
 					(unit 1)
@@
 		(instances
 			(project "omnimarble-driver"
-				(path "/3eaa9588-078e-48af-b393-9dad6bd20142/62eeab2e-1b72-4517-8983-437fbddb3cf0"
+				(path "/4f6b9534-97fd-44ae-b81e-62754cb6cba6/78b057db-20e0-48a6-a5e1-06c21da7677d"
 					(reference "#PWR0007")
 					(unit 1)
