File: hardware/omnimarble-driver/power_input.kicad_sch (KiCad schematic)
At the start: 18 parts, among them J1 24V-IN, Q90 AOD4185, U1 AP63205, U2 78L12, U3 MCP6002

Commit message: Snapshot driver's final validated state before parking as vNext
Fold the last regeneration into the repo so the source is internally consistent
with the already-committed board/BOM (the Q90 diode->MOSFET fix + JLC cart
substitutions previously landed only in the root schematic + board):
- 7 driver schematic sub-sheets, regenerated to carry the final part numbers.
- fab/jlc/ORDER_NOTES.md — final BOM (J2/J5 C707836, R21/R22 C5110275, etc.).
- omnimarble-driver-5-rev-39.ses — the routing session import-clean rebuilds the
  board from; committing it keeps the routed board reproducible while parked.

Timestamp-only gerber/zip churn and scratch (.ses iterations, drc/erc reports,
logs) were left out. Driver stays vNext/on-hold per V0_BENCH_RIG.md.

Co-Authored-By: Claude Opus 4.8 <noreply@anthropic.com>
Parts:
- Q90: LCSC C77317 -> C5371006
Changed lines of the file:
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@@
 		(instances
 			(project "omnimarble-driver"
-				(path "/4f6b9534-97fd-44ae-b81e-62754cb6cba6/78b057db-20e0-48a6-a5e1-06c21da7677d"
+				(path "/e983a447-c241-422e-9650-13442643de66/86c41b1e-95c1-4867-964e-aebfc748663c"
 					(reference "J1")
 					(unit 1)
@@
 		(instances
 			(project "omnimarble-driver"
-				(path "/4f6b9534-97fd-44ae-b81e-62754cb6cba6/78b057db-20e0-48a6-a5e1-06c21da7677d"
+				(path "/e983a447-c241-422e-9650-13442643de66/86c41b1e-95c1-4867-964e-aebfc748663c"
 					(reference "F1")
 					(unit 1)
@@
 			)
 		)
-		(property "LCSC" "C77317"
+		(property "LCSC" "C5371006"
 			(at 100.33 49.53 0)
 			(show_name no)
@@
 		(instances
 			(project "omnimarble-driver"
-				(path "/4f6b9534-97fd-44ae-b81e-62754cb6cba6/78b057db-20e0-48a6-a5e1-06c21da7677d"
+				(path "/e983a447-c241-422e-9650-13442643de66/86c41b1e-95c1-4867-964e-aebfc748663c"
 					(reference "Q90")
 					(unit 1)
@@
 		(instances
 			(project "omnimarble-driver"
-				(path "/4f6b9534-97fd-44ae-b81e-62754cb6cba6/78b057db-20e0-48a6-a5e1-06c21da7677d"
+				(path "/e983a447-c241-422e-9650-13442643de66/86c41b1e-95c1-4867-964e-aebfc748663c"
 					(reference "R1")
 					(unit 1)
@@
 		(instances
 			(project "omnimarble-driver"
-				(path "/4f6b9534-97fd-44ae-b81e-62754cb6cba6/78b057db-20e0-48a6-a5e1-06c21da7677d"
+				(path "/e983a447-c241-422e-9650-13442643de66/86c41b1e-95c1-4867-964e-aebfc748663c"
 					(reference "D1")
 					(unit 1)
@@
 		(instances
 			(project "omnimarble-driver"
-				(path "/4f6b9534-97fd-44ae-b81e-62754cb6cba6/78b057db-20e0-48a6-a5e1-06c21da7677d"
+				(path "/e983a447-c241-422e-9650-13442643de66/86c41b1e-95c1-4867-964e-aebfc748663c"
 					(reference "D90")
 					(unit 1)
@@
 		(instances
 			(project "omnimarble-driver"
-				(path "/4f6b9534-97fd-44ae-b81e-62754cb6cba6/78b057db-20e0-48a6-a5e1-06c21da7677d"
+				(path "/e983a447-c241-422e-9650-13442643de66/86c41b1e-95c1-4867-964e-aebfc748663c"
 					(reference "C1")
 					(unit 1)
@@
 		(instances
 			(project "omnimarble-driver"
-				(path "/4f6b9534-97fd-44ae-b81e-62754cb6cba6/78b057db-20e0-48a6-a5e1-06c21da7677d"
+				(path "/e983a447-c241-422e-9650-13442643de66/86c41b1e-95c1-4867-964e-aebfc748663c"
 					(reference "U1")
 					(unit 1)
@@
 		(instances
 			(project "omnimarble-driver"
-				(path "/4f6b9534-97fd-44ae-b81e-62754cb6cba6/78b057db-20e0-48a6-a5e1-06c21da7677d"
+				(path "/e983a447-c241-422e-9650-13442643de66/86c41b1e-95c1-4867-964e-aebfc748663c"
 					(reference "C2")
 					(unit 1)
@@
 		(instances
 			(project "omnimarble-driver"
-				(path "/4f6b9534-97fd-44ae-b81e-62754cb6cba6/78b057db-20e0-48a6-a5e1-06c21da7677d"
+				(path "/e983a447-c241-422e-9650-13442643de66/86c41b1e-95c1-4867-964e-aebfc748663c"
 					(reference "L1")
 					(unit 1)
@@
 		(instances
 			(project "omnimarble-driver"
-				(path "/4f6b9534-97fd-44ae-b81e-62754cb6cba6/78b057db-20e0-48a6-a5e1-06c21da7677d"
+				(path "/e983a447-c241-422e-9650-13442643de66/86c41b1e-95c1-4867-964e-aebfc748663c"
 					(reference "C3")
 					(unit 1)
@@
 		(instances
 			(project "omnimarble-driver"
-				(path "/4f6b9534-97fd-44ae-b81e-62754cb6cba6/78b057db-20e0-48a6-a5e1-06c21da7677d"
+				(path "/e983a447-c241-422e-9650-13442643de66/86c41b1e-95c1-4867-964e-aebfc748663c"
 					(reference "C4")
 					(unit 1)
@@
 		(instances
 			(project "omnimarble-driver"
-				(path "/4f6b9534-97fd-44ae-b81e-62754cb6cba6/78b057db-20e0-48a6-a5e1-06c21da7677d"
+				(path "/e983a447-c241-422e-9650-13442643de66/86c41b1e-95c1-4867-964e-aebfc748663c"
 					(reference "U2")
 					(unit 1)
@@
 		(instances
 			(project "omnimarble-driver"
-				(path "/4f6b9534-97fd-44ae-b81e-62754cb6cba6/78b057db-20e0-48a6-a5e1-06c21da7677d"
+				(path "/e983a447-c241-422e-9650-13442643de66/86c41b1e-95c1-4867-964e-aebfc748663c"
 					(reference "C5")
 					(unit 1)
@@
 		(instances
 			(project "omnimarble-driver"
-				(path "/4f6b9534-97fd-44ae-b81e-62754cb6cba6/78b057db-20e0-48a6-a5e1-06c21da7677d"
+				(path "/e983a447-c241-422e-9650-13442643de66/86c41b1e-95c1-4867-964e-aebfc748663c"
 					(reference "C6")
 					(unit 1)
@@
 		(instances
 			(project "omnimarble-driver"
-				(path "/4f6b9534-97fd-44ae-b81e-62754cb6cba6/78b057db-20e0-48a6-a5e1-06c21da7677d"
+				(path "/e983a447-c241-422e-9650-13442643de66/86c41b1e-95c1-4867-964e-aebfc748663c"
 					(reference "R2")
 					(unit 1)
@@
 		(instances
 			(project "omnimarble-driver"
-				(path "/4f6b9534-97fd-44ae-b81e-62754cb6cba6/78b057db-20e0-48a6-a5e1-06c21da7677d"
+				(path "/e983a447-c241-422e-9650-13442643de66/86c41b1e-95c1-4867-964e-aebfc748663c"
 					(reference "R3")
 					(unit 1)
@@
 		(instances
 			(project "omnimarble-driver"
-				(path "/4f6b9534-97fd-44ae-b81e-62754cb6cba6/78b057db-20e0-48a6-a5e1-06c21da7677d"
+				(path "/e983a447-c241-422e-9650-13442643de66/86c41b1e-95c1-4867-964e-aebfc748663c"
 					(reference "U3")
 					(unit 2)
@@
 		(instances
 			(project "omnimarble-driver"
-				(path "/4f6b9534-97fd-44ae-b81e-62754cb6cba6/78b057db-20e0-48a6-a5e1-06c21da7677d"
+				(path "/e983a447-c241-422e-9650-13442643de66/86c41b1e-95c1-4867-964e-aebfc748663c"
 					(reference "#FLG0001")
 					(unit 1)
@@
 		(instances
 			(project "omnimarble-driver"
-				(path "/4f6b9534-97fd-44ae-b81e-62754cb6cba6/78b057db-20e0-48a6-a5e1-06c21da7677d"
+				(path "/e983a447-c241-422e-9650-13442643de66/86c41b1e-95c1-4867-964e-aebfc748663c"
 					(reference "#FLG0002")
 					(unit 1)
@@
 		(instances
 			(project "omnimarble-driver"
-				(path "/4f6b9534-97fd-44ae-b81e-62754cb6cba6/78b057db-20e0-48a6-a5e1-06c21da7677d"
+				(path "/e983a447-c241-422e-9650-13442643de66/86c41b1e-95c1-4867-964e-aebfc748663c"
 					(reference "#PWR0003")
 					(unit 1)
@@
 		(instances
 			(project "omnimarble-driver"
-				(path "/4f6b9534-97fd-44ae-b81e-62754cb6cba6/78b057db-20e0-48a6-a5e1-06c21da7677d"
+				(path "/e983a447-c241-422e-9650-13442643de66/86c41b1e-95c1-4867-964e-aebfc748663c"
 					(reference "#FLG0004")
 					(unit 1)
@@
 		(instances
 			(project "omnimarble-driver"
-				(path "/4f6b9534-97fd-44ae-b81e-62754cb6cba6/78b057db-20e0-48a6-a5e1-06c21da7677d"
+				(path "/e983a447-c241-422e-9650-13442643de66/86c41b1e-95c1-4867-964e-aebfc748663c"
 					(reference "#FLG0005")
 					(unit 1)
@@
 		(instances
 			(project "omnimarble-driver"
-				(path "/4f6b9534-97fd-44ae-b81e-62754cb6cba6/78b057db-20e0-48a6-a5e1-06c21da7677d"
+				(path "/e983a447-c241-422e-9650-13442643de66/86c41b1e-95c1-4867-964e-aebfc748663c"
 					(reference "#FLG0006")
 					(unit 1)
@@
 		(instances
 			(project "omnimarble-driver"
-				(path "/4f6b9534-97fd-44ae-b81e-62754cb6cba6/78b057db-20e0-48a6-a5e1-06c21da7677d"
+				(path "/e983a447-c241-422e-9650-13442643de66/86c41b1e-95c1-4867-964e-aebfc748663c"
 					(reference "#PWR0007")
 					(unit 1)
